File: PCB/ZORRO-LAN-IDE-CP-V2E.sch (EAGLE design)
At the start: 41 parts, among them CN1 ZORROII_EDGE_ROUND_CONTACTS, IC1 OLIMEX_ENC, IC2 XC95288XL-TQ144, IC3 74HCT245PW, IC4 74HCT245PW, IC5 74HCT245PW, IC7 LD117AS33TR, IC8 AM29F010J-SOCKET

Commit message: Clean up and driver update
Parts:
- removed INT6/INT2: (no value), jumper:SJ2W
- added AUTOBOOT_ON: (no value), jumper:JP1E
- added C1, C13, C18, C3, C4, C6, C7, C8: 100nF, rcl:C-EUC0805K
- added C19: 10u, rcl:C-EUC1206K
- added C24, C25: 27p, rcl:C-EUC0805K
- added C26, C27: 6.8n, rcl:C-EUC0805K
- added C28, C33: 10n, rcl:C-EUC0805K
- added C29, C30, C32: 100n, rcl:C-EUC0603K
- added C31: 47u, rcl:C-EUC1210K
- added C5: 47uF, rcl:C-EUC1206K
- added CN2: A1200-CLOCKPORT, Amiga:A1200-CLOCKPORT
- added Q1: 25MHz, crystal:CRYSTALHC18U-V
- added Q2: 25MHz, crystal:CRYSTALHC49UP
- added R10, R11: 1K, rcl:R-EU_R0805
- added R12: 3.3k, rcl:R-EU_R0603
- added R13: 12k, rcl:R-EU_R0603
- added R14: 180, rcl:R-EU_R0603
- added R15, R16, R17, R18: 49.9, rcl:R-EU_R0603
- added R19: 10, rcl:R-EU_R0603
- added SJ2: (no value), jumper:SJ
- added SV1: (no value), con-ml:ML14
- added X1: SI-50170, con-stewart:SI-50170
- C10, C11, C12, C9: value (none) -> 100n
- C20, C21: device rcl:C-EUC0805K -> rcl:C-EUC1210K
- IC1: value OLIMEX_ENC -> ENC624J600; device OLIMEX-ENJ:OLIMEX_ENC -> OLIMEX-ENJ:ENC624J600
- IC7: value LD117AS33TR -> LD117ADT33TR; device v-reg:LD117AS33TR -> v-reg:LD117ADT33TR
- IC8: value AM29F010J-SOCKET -> AM29F010S; device am29-memory:AM29F010J-SOCKET -> am29-memory:AM29F010S
- JP1: device pinhead-2:PINHD-1X02_2.54-S -> jumper:JP1E
- R1: value 330 -> 4.7k
- R4: value 100k -> 390
- R6: value 330 -> 180
- renumbered AUTOBOOT_OFF to IDE_OFF
Connections:
- removed net INT_OUT: IC2.P$32-FB3MC14/GCK2, INT6/INT2.2, R9.2
- removed net N$1: LEDA.1, R1.2
- removed net N$2: LEDB.1, R6.2
- removed net ROM_B2: IC2.P$70-FB11MC17, IC8NC1.NC
- removed net ROM_B3: IC2.P$71-FB13MC02, IC8NC2.NC
- removed net ROM_WE: IC2.P$34-FB5MC02, IC8G$1.WE/
- removed net VCC: JP1.2
- new net CP_CS: CN2.!SPARE-CS, IC2.P$34-FB5MC02
- new net CP_IRQ: CN2.!INT6, IC2.P$31-FB3MC12, R11.2
- new net CP_RD: CN2.!IORD, IC2.P$71-FB13MC02
- new net CP_WE: CN2.!IOWR, IC2.P$70-FB11MC17
- new net DOE: CN1.DOE, IC2.P$38-FB5MC08/GCK3
- new net LEDAC: LEDA.2, R14.1, SV1.2, X1.C
- new net LEDBC: LEDB.2, R6.1, SV1.14, X1.C1
- new net N$3: CN2.!RTC-CS, CN2.!RTC-DS, R10.2
- new net N$4: C19.1, IC1.VCAP
- new net N$5: R13.1, R4.2
- new net N$6: IC1.RBIAS, R4.1
- new net N$8: C25.1, IC1.OSC_I, Q1.1, Q2.1
- new net N$9: C24.1, IC1.OSC_O, Q1.2, Q2.2
- new net RCT: C33.1, R15.1, R16.1, SJ2.2, X1.RCT
- new net RD+: C26.2, SV1.6
- new net RD++: SV1.4, X1.RD+
- new net RD-: C27.2, SV1.5
- new net RD--: SJ2.1, SV1.3, X1.RD-
- new net ROM_CE: AUTOBOOT_ON.2, IC8G$1.!CE, R1.2
- new net TCT: C28.2, R19.1, SV1.11, X1.TCT
- new net TD+: SV1.8, X1.TD+
- new net TD-: SV1.7, X1.TD-
- new net TPIN+: C26.1, IC1.TPIN+, R16.2
- new net TPIN-: C27.1, IC1.TPIN-, R15.2
- new net TPOUT+: IC1.TPOUT+, R17.1, SV1.10
- new net TPOUT-: IC1.TPOUT-, R18.1, SV1.9
- net +3V3: now also C1.2, C13.2, C18.2, C29.1, C3.2, C30.2, C32.1, C6.2, C7.2, C8.2, IC1.PSPCFG2, IC1.VDD, IC1.VDD@2, IC1.VDD@3, IC1.VDD_OSC, IC1.VDD_PLL, IC1.VDD_RX, IC1.VDD_TX, R17.2, R18.2, R19.2; no longer IC1EXT1.3V3@1, IC1EXT1.3V3@2, IC1EXT1.3V3@3, IC1EXT2.3V3@1, IC1EXT2.3V3@2
- net +5V: now also C31.1, C4.2, C5.1, CN2.+5V, IC8G$1.WE/, IC8NC1.NC, IC8NC2.NC, JP1.2, R1.1, R10.1, R11.1, R2.1, R5.1, RN1D.2, SV2.4; no longer IDE_OFF.1, SV2.1
- net CLK_EXT: now also IC1.CLK_OUT; no longer IC1EXT1.CLK_O
- net D0: no longer IC3A.A2, IC8G$1.O0
- net D1: no longer IC3A.A4, IC8G$1.O1
- net D10: no longer IC4A.A3
- net D11: no longer IC4A.A1
- net D12: no longer IC3A.A7
- net D13: no longer IC3A.A5
- net D14: no longer IC3A.A3
- net D15: no longer IC3A.A1
- net D2: no longer IC3A.A6, IC8G$1.O2
- net D3: no longer IC3A.A8, IC8G$1.O3
- net D4: no longer IC4A.A2, IC8G$1.O4
- net D5: no longer IC4A.A4, IC8G$1.O5
- net D6: no longer IC4A.A6, IC8G$1.O6
- net D7: no longer IC4A.A8, IC8G$1.O7
- net D8: no longer IC4A.A7
- net D9: no longer IC4A.A5
- net DQ0: now also CN2.D16, IC1.AD0, IC3A.A2, IC8G$1.O0; no longer IC1EXT2.AD0
- net DQ1: now also CN2.D17, IC1.AD1, IC3A.A4, IC8G$1.O1; no longer IC1EXT2.AD1
- net DQ10: now also IC1.AD10, IC4A.A3; no longer IC1EXT2.AD10
- net DQ11: now also IC1.AD11, IC4A.A1; no longer IC1EXT2.AD11
- net DQ12: now also IC1.AD12, IC3A.A7; no longer IC1EXT2.AD12
- net DQ13: now also IC1.AD13, IC3A.A5; no longer IC1EXT2.AD13
- net DQ14: now also IC1.AD14, IC3A.A3; no longer IC1EXT2.AD14
- net DQ15: now also IC1.AD15, IC3A.A1; no longer IC1EXT2.AD15
- net DQ2: now also CN2.D18, IC1.AD2, IC3A.A6, IC8G$1.O2; no longer IC1EXT2.AD2
- net DQ3: now also CN2.D19, IC1.AD3, IC3A.A8, IC8G$1.O3; no longer IC1EXT2.AD3
- net DQ4: now also CN2.D20, IC1.AD4, IC4A.A2, IC8G$1.O4; no longer IC1EXT2.AD4
- net DQ5: now also CN2.D21, IC1.AD5, IC4A.A4, IC8G$1.O5; no longer IC1EXT2.AD5
- net DQ6: now also CN2.D22, IC1.AD6, IC4A.A6, IC8G$1.O6; no longer IC1EXT2.AD6
- net DQ7: now also CN2.D23, IC1.AD7, IC4A.A8, IC8G$1.O7; no longer IC1EXT2.AD7
- net DQ8: now also IC1.AD8, IC4A.A7; no longer IC1EXT2.AD8
- net DQ9: now also IC1.AD9, IC4A.A5; no longer IC1EXT2.AD9
- net GND: now also AUTOBOOT_ON.1, C1.1, C13.1, C18.1, C19.2, C24.2, C25.2, C28.1, C29.2, C3.1, C30.1, C31.2, C32.2, C33.2, C4.1, C5.2, C6.1, C7.1, C8.1, CN2.GND@1, CN2.GND@2, IC1.A14/PSPCFG1, IC1.PSPCFG3, IC1.PSPCFG4, IC1.VSS, IC1.VSS@2, IC1.VSS_OSC, IC1.VSS_PLL, IC1.VSS_RX, IC1.VSS_TX, IC1.VSS_TX@2, IDE_OFF.1, R12.1, R13.2, R14.2, R6.2, SV1.12, X1.C_GND, X1.S1, X1.S2; no longer IC1EXT1.GND@1, IC1EXT1.GND@2, IC1EXT1.GND@3, IC1EXT2.GND@1, IC1EXT2.GND@2, IC8G$1.!CE, R1.1, R2.1, R4.1, R5.1, R6.1, SV2.4, SV2.6, SV2.8
- net IDE_IRQ: no longer IC2.P$31-FB3MC12
- net IDE_RST: now also CN2.!RESET
- net INT2: now also IC2.P$32-FB3MC14/GCK2, R9.2; no longer INT6/INT2.1
- net INT6: no longer INT6/INT2.3
- net LAN_A0: now also IC1.A0; no longer IC1EXT1.A0
- net LAN_A1: now also IC1.A1; no longer IC1EXT1.A1
- net LAN_A10: now also IC1.A10; no longer IC1EXT1.A10
- net LAN_A11: now also IC1.A11; no longer IC1EXT1.A11
- net LAN_A12: now also IC1.A12; no longer IC1EXT1.A12
- net LAN_A13: now also IC1.A13; no longer IC1EXT1.A13
- net LAN_A2: now also IC1.A2; no longer IC1EXT1.A2
- net LAN_A3: now also CN2.A2, IC1.A3; no longer IC1EXT1.A3
- net LAN_A4: now also CN2.A3, IC1.A4; no longer IC1EXT1.A4
- net LAN_A5: now also CN2.A4, IC1.A5; no longer IC1EXT1.A5
- net LAN_A6: now also CN2.A5, IC1.A6; no longer IC1EXT1.A6
- net LAN_A7: now also IC1.A7; no longer IC1EXT1.A7
- net LAN_A8: now also IC1.A8; no longer IC1EXT1.A8
- net LAN_A9: now also IC1.A9; no longer IC1EXT1.A9
- net LAN_CFG1: no longer IC1EXT1.PCFG1
- net LAN_CFG3: no longer IC1EXT1.PCFG3
- net LAN_CFG4: no longer IC1EXT2.PCGF4
- net LAN_CGF2: no longer IC1EXT1.PCFG2
- net LAN_CS: now also IC1.!CS; no longer IC1EXT2._CS
- net LAN_EN: now also IC1.WRL; no longer IC1EXT2.EN
- net LAN_INT: now also IC1.!INT!/SPISEL, R12.2; no longer IC1EXT2.INT, R4.2
- net LAN_RD: now also IC1.!RW; no longer IC1EXT2.RD
- net LAN_WRH: now also IC1.WRH; no longer IC1EXT2.WRH
- net LEDA: now also IC1.LED_A, LEDA.1, SV1.1, X1.A; no longer IC1EXT1.LEDA, LEDA.2
- net LEDB: now also IC1.LED_B, LEDB.1, SV1.13, X1.A1; no longer IC1EXT1.LEDB, LEDB.2
- net TCK: now also SV2.1; no longer SV2.9
- net TDI: now also SV2.9; no longer SV2.5
- net TMS: now also SV2.5; no longer SV2.7
Other:
- note added: "<- LAN-port adresses are shifted by one! Amiga_A1 = LAN_A0"
